Commit message: Completed PID control algorithm

File: diffdrive_ws/install/diffdrive_description/share/diffdrive_description/urdf/common_properties.xacro (robot description, xacro)
@@ -1 +1,45 @@
-/home/robomango/workspace/MangoMobileRobot/diffdrive_ws/src/diffdrive_description/urdf/common_properties.xacro
+<?xml version="1.0"?>
+<robot xmlns:xacro="http://www.ros.org/wiki/xacro">
+    <material name="blue">
+        <color rgba="0 0 0.8 1"/>
+    </material>
+    <material name="grey">
+        <color rgba="0.1 0.1 0.1 1"/>
+    </material>
+    <material name="black">
+        <color rgba="0 0 0 1"/>
+    </material>
+    <material name="white">
+        <color rgba="1 1 1 1"/>
+    </material>
+    <xacro:macro name="box_inertia" params="m l w h xyz rpy">
+        <inertial>
+            <origin xyz="${xyz}" rpy="${rpy}" />
+            <mass value ="${m}"/>
+            <inertia ixx="${(m/12) * (l*l + h*h)}" ixy="0" ixz="0"
+                iyy="${(m/12) * (w*w + l*l)}" iyz="0"
+                izz="${(m/12) * (w*w + h*h)}" >
+            </inertia>
+        </inertial>
+    </xacro:macro>
+    <xacro:macro name="cylinder_inertia" params="m r h xyz rpy">
+        <inertial>
+            <origin xyz="${xyz}" rpy="${rpy}" />
+            <mass value ="${m}"/>
+            <inertia ixx="${(m/12) * (3*r*r + h*h)}" ixy="0" ixz="0"
+                iyy="${(m/12) * (3*r*r + h*h)}" iyz="0"
+                izz="${(m/2) * (r*r)}" >
+            </inertia>
+        </inertial>
+    </xacro:macro>
+    <xacro:macro name="sphere_inertia" params="m r xyz rpy">
+        <inertial>
+            <origin xyz="${xyz}" rpy="${rpy}" />
+            <mass value="${m}"/>
+            <inertia ixx="${(2/5)*m*r*r}" ixy="0" ixz="0"
+                iyy="${(2/5)*m*r*r}" iyz="0"
+                izz="0">
+            </inertia>
+        </inertial>
+    </xacro:macro>
+</robot>

File: diffdrive_ws/install/diffdrive_description/share/diffdrive_description/urdf/mobile_base.xacro (robot description, xacro)
@@ -1 +1,87 @@
-/home/robomango/workspace/MangoMobileRobot/diffdrive_ws/src/diffdrive_description/urdf/mobile_base.xacro
+<?xml version="1.0"?>
+<robot xmlns:xacro="http://www.ros.org/wiki/xacro">
+    <xacro:property name="base_length" value="0.125"/>
+    <xacro:property name="base_width" value="0.08"/>
+    <xacro:property name="base_height" value="0.02"/>
+    <xacro:property name="wheel_radius" value="0.02"/>
+    <xacro:property name="wheel_length" value="0.017"/>
+    <xacro:property name="caster_radius" value="${wheel_radius / 2.0}"/>
+    <link name="base_footprint"/>
+    <link name="base_link">
+        <visual>
+            <geometry>
+                <box size="${base_length} ${base_width} ${base_height}"/>
+            </geometry>
+            <origin xyz="0 0 ${base_height / 2.0}" rpy="0 0 0"/>
+            <material name="white"/>
+        </visual>
+        <xacro:box_inertia m="5.0" l="${2*base_length}" w="${2*base_width}" h="${2*base_height}"
+         xyz="0 0 ${2*base_height / 2.0}" rpy="0 0 0" />
+        <collision>
+            <geometry>
+                <box size="${base_length} ${base_width} ${base_height}"/>
+            </geometry>
+            <origin xyz="0 0 ${base_height / 2.0}" rpy="0 0 0"/>
+        </collision>
+    </link>
+    <xacro:macro name="wheel_link" params="prefix">
+        <link name="${prefix}_wheel_link">
+            <visual>
+                <geometry>
+                    <cylinder radius="${wheel_radius}" length="${wheel_length}"/>
+                </geometry>
+                <origin xyz="0 0 0" rpy="${pi/2.0} 0 0"/>
+                <material name ="grey"/>
+            </visual>
+            <xacro:cylinder_inertia m="1.0" r="${2*wheel_radius}" h="${2*wheel_length}" xyz="0 0 0" rpy="${pi/2.0} 0 0"/>
+            <collision>
+                <geometry>
+                    <cylinder radius="${wheel_radius}" length="${wheel_length}"/>
+                </geometry>
+                <origin xyz="0 0 0" rpy="${pi/2.0} 0 0"/>
+            </collision>
+        </link>
+    </xacro:macro>
+    <xacro:wheel_link prefix="left"/>
+    <xacro:wheel_link prefix="right"/>
+    <link name="caster_wheel_link">
+        <visual>
+            <geometry>
+                <sphere radius="${caster_radius}"/>
+            </geometry>
+            <origin xyz="0 0 0" rpy="0 0 0"/>
+            <material name="grey"/>
+        </visual>
+        <xacro:sphere_inertia m="0.5" r="${2*caster_radius}" xyz="0 0 0" rpy="0 0 0" />
+        <collision>
+            <geometry>
+                <sphere radius="${caster_radius}"/>
+            </geometry>
+            <origin xyz="0 0 0" rpy="0 0 0"/>
+        </collision>
+    </link>
+    <joint name="base_joint" type="fixed">
+        <parent link="base_footprint"/>
+        <child link="base_link"/>
+        <origin xyz="0 0 ${wheel_radius}" rpy="0 0 0"/>
+    </joint>
+    <joint name="base_right_wheel_joint" type="continuous">
+        <parent link="base_link"/>
+        <child link="right_wheel_link"/>
+        <origin xyz="${-base_length / 4.0} ${-((base_width / 2.0) + (wheel_length/2.0))} 0" rpy="0 0 0"/>
+        <axis xyz="0 1 0"/>
+        <limit velocity="100" effort="100"/>
+    </joint>
+    <joint name="base_left_wheel_joint" type="continuous">
+        <parent link="base_link"/>
+        <child link="left_wheel_link"/>
+        <origin xyz="${-base_length / 4.0} ${(base_width / 2.0) + (wheel_length/2.0)} 0" rpy="0 0 0"/>
+        <axis xyz="0 1 0"/>
+        <limit velocity="100" effort="100"/>
+    </joint>
+    <joint name="base_caster_wheel_joint" type="fixed">
+        <parent link="base_link"/>
+        <child link="caster_wheel_link"/>
+        <origin xyz="${base_length / 3.0} 0 ${-caster_radius}" rpy="0 0 0"/>
+    </joint>
+</robot>

File: diffdrive_ws/install/diffdrive_description/share/diffdrive_description/urdf/my_robot.urdf.xacro (robot description, xacro)
@@ -1 +1,5 @@
-/home/robomango/workspace/MangoMobileRobot/diffdrive_ws/src/diffdrive_description/urdf/my_robot.urdf.xacro
+<?xml version="1.0"?>
+<robot name="Nav2bot" xmlns:xacro="http://www.ros.org/wiki/xacro">
+    <xacro:include filename="common_properties.xacro"/>
+    <xacro:include filename="mobile_base.xacro"/>
+</robot>
